File: pcb/adelheid.kicad_sch (KiCad schematic)
At the start: 35 parts, among them J1 USB_C_Receptacle_USB2.0, J2 Conn_01x04, J8 Conn_01x06, Q1 2N7002, U1 USBLC6-2SC6, U2 ATmega32U4-AU, Y1 Crystal_GND24

Commit message: changes key footprints to hotswap + SMD LEDs
Parts:
- Y1: footprint Crystals:Crystal_SMD_SeikoEpson_FA238-4pin_3.2x2.5mm_HandSoldering -> Crystal:Crystal_SMD_SeikoEpson_FA238-4Pin_3.2x2.5mm
Changed lines of the file:
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@@
 			)
 		)
-		(property "Footprint" "Crystals:Crystal_SMD_SeikoEpson_FA238-4pin_3.2x2.5mm_HandSoldering"
+		(property "Footprint" "Crystal:Crystal_SMD_SeikoEpson_FA238-4Pin_3.2x2.5mm"
 			(at 63.5 92.71 0)
 			(effects
