File: pcb/matrix.kicad_sch (KiCad schematic)
At the start: 242 parts, among them SW1 Rotary_Encoder_Switch

Commit message: fix cutouts (encoder + tab + backspace)
Parts:
- MX65: value ~ -> (none)
- SW1: footprint Rotary_Encoder:RotaryEncoder_Alps_EC11E-Switch_Vertical_H20mm -> adelheid:RotaryEncoder_Alps_EC11E-Switch_Vertical_H20mm
