File: macro-pad/matrix.kicad_sch (KiCad schematic)
At the start: 53 parts, among them SW1 Rotary_Encoder_Switch

Commit message: add case plates generation
Parts:
- MX1, MX10, MX12, MX13, MX14, MX15, MX16, MX18, MX2, MX3, MX4, MX7, MX8, MX9: footprint ai03-MX_only:MXOnly-1U -> ai03-MX_only:MXOnly-1U-Hotswap-Antishear-Led-SMD
- MX20, MX22, MX5: footprint ai03-MX_only:MXOnly-2U -> ai03-MX_only:MXOnly-2U-Hotswap-Antishear-Led-SMD
Changed lines of the file:
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@@
 (kicad_sch
-	(version 20231120)
+	(version 20250114)
 	(generator "eeschema")
-	(generator_version "8.0")
+	(generator_version "9.0")
 	(paper "A3")
 	(junction
@@
 		(shape input)
 		(at 81.28 53.34 180)
-		(fields_autoplaced yes)
 		(effects
 			(font
@@
 		(shape input)
 		(at 321.31 201.93 0)
-		(fields_autoplaced yes)
 		(effects
 			(font
@@
 		(shape tri_state)
 		(at 354.33 38.1 90)
-		(fields_autoplaced yes)
 		(effects
 			(font
@@
 		(shape tri_state)
 		(at 297.18 38.1 90)
-		(fields_autoplaced yes)
 		(effects
 			(font
@@
 		(shape tri_state)
 		(at 182.88 38.1 90)
-		(fields_autoplaced yes)
 		(effects
 			(font
@@
 		(shape tri_state)
 		(at 106.68 38.1 90)
-		(fields_autoplaced yes)
 		(effects
 			(font
@@
 		(shape tri_state)
 		(at 220.98 38.1 90)
-		(fields_autoplaced yes)
 		(effects
 			(font
@@
 		(shape tri_state)
 		(at 144.78 38.1 90)
-		(fields_autoplaced yes)
 		(effects
 			(font
@@
 		(shape tri_state)
 		(at 278.13 38.1 90)
-		(fields_autoplaced yes)
 		(effects
 			(font
@@
 		(shape tri_state)
 		(at 80.01 137.16 180)
-		(fields_autoplaced yes)
 		(effects
 			(font
@@
 		(shape tri_state)
 		(at 80.01 113.03 180)
-		(fields_autoplaced yes)
 		(effects
 			(font
@@
 		(shape tri_state)
 		(at 373.38 38.1 90)
-		(fields_autoplaced yes)
 		(effects
 			(font
@@
 		(shape tri_state)
 		(at 201.93 38.1 90)
-		(fields_autoplaced yes)
 		(effects
 			(font
@@
 		(shape tri_state)
 		(at 80.01 88.9 180)
-		(fields_autoplaced yes)
 		(effects
 			(font
@@
 		(shape tri_state)
 		(at 259.08 38.1 90)
-		(fields_autoplaced yes)
 		(effects
 			(font
@@
 		(shape input)
 		(at 321.31 207.01 0)
-		(fields_autoplaced yes)
 		(effects
 			(font
@@
 		(shape tri_state)
 		(at 125.73 38.1 90)
-		(fields_autoplaced yes)
 		(effects
 			(font
@@
 		(shape tri_state)
 		(at 80.01 64.77 180)
-		(fields_autoplaced yes)
 		(effects
 			(font
@@
 		(shape tri_state)
 		(at 316.23 38.1 90)
-		(fields_autoplaced yes)
 		(effects
 			(font
@@
 		(shape tri_state)
 		(at 240.03 38.1 90)
-		(fields_autoplaced yes)
 		(effects
 			(font
@@
 		(shape tri_state)
 		(at 335.28 38.1 90)
-		(fields_autoplaced yes)
 		(effects
 			(font
@@
 		(shape tri_state)
 		(at 163.83 38.1 90)
-		(fields_autoplaced yes)
 		(effects
 			(font
@@
 		(shape tri_state)
 		(at 80.01 161.29 180)
-		(fields_autoplaced yes)
 		(effects
 			(font
@@
 		(shape bidirectional)
 		(at 80.01 185.42 180)
-		(fields_autoplaced yes)
 		(effects
 			(font
@@
 			)
 		)
-		(property "Footprint" "ai03-MX_only:MXOnly-1U"
+		(property "Footprint" "ai03-MX_only:MXOnly-1U-Hotswap-Antishear-Led-SMD"
 			(at 86.995 52.705 0)
 			(effects
@@
 			)
 		)
-		(property "Footprint" "ai03-MX_only:MXOnly-1U"
+		(property "Footprint" "ai03-MX_only:MXOnly-1U-Hotswap-Antishear-Led-SMD"
 			(at 106.045 52.705 0)
 			(effects
@@
 			)
 		)
-		(property "Footprint" "ai03-MX_only:MXOnly-1U"
+		(property "Footprint" "ai03-MX_only:MXOnly-1U-Hotswap-Antishear-Led-SMD"
 			(at 125.095 52.705 0)
 			(effects
@@
 			)
 		)
-		(property "Footprint" "ai03-MX_only:MXOnly-1U"
+		(property "Footprint" "ai03-MX_only:MXOnly-1U-Hotswap-Antishear-Led-SMD"
 			(at 144.145 52.705 0)
 			(effects
@@
 			)
 		)
-		(property "Footprint" "ai03-MX_only:MXOnly-2U"
+		(property "Footprint" "ai03-MX_only:MXOnly-2U-Hotswap-Antishear-Led-SMD"
 			(at 86.995 149.225 0)
 			(effects
@@
 			)
 		)
-		(property "Footprint" "ai03-MX_only:MXOnly-1U"
+		(property "Footprint" "ai03-MX_only:MXOnly-1U-Hotswap-Antishear-Led-SMD"
 			(at 125.095 76.835 0)
 			(effects
@@
 			)
 		)
-		(property "Footprint" "ai03-MX_only:MXOnly-1U"
+		(property "Footprint" "ai03-MX_only:MXOnly-1U-Hotswap-Antishear-Led-SMD"
 			(at 86.995 76.835 0)
 			(effects
@@
 			)
 		)
-		(property "Footprint" "ai03-MX_only:MXOnly-1U"
+		(property "Footprint" "ai03-MX_only:MXOnly-1U-Hotswap-Antishear-Led-SMD"
 			(at 106.045 76.835 0)
 			(effects
@@
 			)
 		)
-		(property "Footprint" "ai03-MX_only:MXOnly-2U"
+		(property "Footprint" "ai03-MX_only:MXOnly-2U-Hotswap-Antishear-Led-SMD"
 			(at 144.145 100.965 0)
 			(effects
@@
 			)
 		)
-		(property "Footprint" "ai03-MX_only:MXOnly-1U"
+		(property "Footprint" "ai03-MX_only:MXOnly-1U-Hotswap-Antishear-Led-SMD"
 			(at 125.095 100.965 0)
 			(effects
@@
 			)
 		)
-		(property "Footprint" "ai03-MX_only:MXOnly-1U"
+		(property "Footprint" "ai03-MX_only:MXOnly-1U-Hotswap-Antishear-Led-SMD"
 			(at 86.995 100.965 0)
 			(effects
@@
 			)
 		)
-		(property "Footprint" "ai03-MX_only:MXOnly-1U"
+		(property "Footprint" "ai03-MX_only:MXOnly-1U-Hotswap-Antishear-Led-SMD"
 			(at 106.045 100.965 0)
 			(effects
@@
 			)
 		)
-		(property "Footprint" "ai03-MX_only:MXOnly-1U"
+		(property "Footprint" "ai03-MX_only:MXOnly-1U-Hotswap-Antishear-Led-SMD"
 			(at 125.095 125.095 0)
 			(effects
@@
 			)
 		)
-		(property "Footprint" "ai03-MX_only:MXOnly-1U"
+		(property "Footprint" "ai03-MX_only:MXOnly-1U-Hotswap-Antishear-Led-SMD"
 			(at 106.045 125.095 0)
 			(effects
@@
 			)
 		)
-		(property "Footprint" "ai03-MX_only:MXOnly-2U"
+		(property "Footprint" "ai03-MX_only:MXOnly-2U-Hotswap-Antishear-Led-SMD"
 			(at 144.145 125.095 0)
 			(effects
@@
 			)
 		)
-		(property "Footprint" "ai03-MX_only:MXOnly-1U"
+		(property "Footprint" "ai03-MX_only:MXOnly-1U-Hotswap-Antishear-Led-SMD"
 			(at 125.095 149.225 0)
 			(effects
@@
 			)
 		)
-		(property "Footprint" "ai03-MX_only:MXOnly-1U"
+		(property "Footprint" "ai03-MX_only:MXOnly-1U-Hotswap-Antishear-Led-SMD"
 			(at 86.995 125.095 0)
 			(effects

Commit message: update lib for correct cad generation
Parts:
- SW1: footprint Rotary_Encoder:RotaryEncoder_Alps_EC11E-Switch_Vertical_H20mm -> keeb-conn:RotaryEncoder_Alps_EC11E-Switch_Vertical_H20mm
Changed lines of the file:
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@@
 			)
 		)
-		(property "Footprint" "Rotary_Encoder:RotaryEncoder_Alps_EC11E-Switch_Vertical_H20mm"
+		(property "Footprint" "keeb-conn:RotaryEncoder_Alps_EC11E-Switch_Vertical_H20mm"
 			(at 309.88 208.534 0)
 			(effects
