File: macro-pad/macro-pad.kicad_pcb (KiCad board)
At the start: 2 copper layers, 100 x 100 mm, 82 parts, among them J1 USB_C_Receptacle_USB2.0, J2 Conn_01x04, J8 Conn_01x06, Q1 2N7002, SW1 Rotary_Encoder_Switch, U1 USBLC6-2SC6, U2 ATmega32U4-AU, Y1 Crystal_GND24

Commit message: optimized python scripts
Parts:
- moved R7 0.40 mm to (117.5, 48.7)
Changed lines of the file:
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@@
 	(footprint "Resistor_SMD:R_0603_1608Metric"
 		(layer "B.Cu")
-		(at 117.5 48.3 -90)
+		(at 117.5 48.7 -90)
 		(descr "Resistor SMD 0603 (1608 Metric), square (rectangular) end terminal, IPC-7351 nominal, (Body size source: IPC-SM-782 page 72, https://www.pcb-3d.com/wordpress/wp-content/uploads/ipc-sm-782a_amendment_1_and_2.pdf), generated with kicad-footprint-generator")
 		(tags "resistor")
@@
 		)
 		(fp_line
-			(start -5.32 -4.15)
-			(end 5.32 -4.15)
-			(stroke
-				(width 0.05)
-				(type solid)
-			)
-			(layer "B.CrtYd")
-		)
-		(fp_line
-			(start -5.32 5.27)
-			(end -5.32 -4.15)
-			(stroke
-				(width 0.05)
-				(type solid)
-			)
-			(layer "B.CrtYd")
-		)
-		(fp_line
-			(start -5.32 5.27)
-			(end 5.32 5.27)
-			(stroke
-				(width 0.05)
-				(type solid)
-			)
-			(layer "B.CrtYd")
-		)
-		(fp_line
-			(start 5.32 5.27)
-			(end 5.32 -4.15)
-			(stroke
-				(width 0.05)
-				(type solid)
-			)
-			(layer "B.CrtYd")
-		)
-		(fp_line
